Commit message: first commit, belum lengkap

File: urdf/cobot.urdf (robot description, URDF)
Before this commit: robot cobot, 12 links, 11 joints
Links:
- removed link in_left_grip
- removed link left_gripper
- removed link out_left_grip
- removed link out_right_grip
- removed link right_gripper
Joints:
- removed joint joint_link5_to_in_left_grip
- removed joint joint_link5_to_out_left_grip
- removed joint joint_link5_to_out_right_grip
- removed joint joint_out_left_grip_to_left_gripper
- removed joint joint_out_right_grip_to_right_gripper
- joint joint_base_link_to_link1: axis -0.0 -0.0 1.0 -> 0 0 1; origin xyz=0.0 0.0 0.05675 rpy=0 0 0 -> xyz=0 0 0.05675 rpy=0 0 0
- joint joint_link1_to_link2: axis -0.000506 -1.0 -0.0 -> 0 0 1; origin xyz=0.01392 -7e-06 0.070276 rpy=0 0 0 -> xyz=0.01392 0 0.070276 rpy=1.5708 -1.5708 0
- joint joint_link2_to_link3: axis 0.000506 1.0 0.0 -> 0 0 -1; origin xyz=-1.5e-05 0.0 0.12 rpy=0 0 0 -> xyz=0.12 0 0 rpy=0 0 0
- joint joint_link3_to_link4: axis -0.0024 1e-06 0.999997 -> 0 0 1; origin xyz=-0.00041 0.010544 0.08975 rpy=0 0 0 -> xyz=0.08975 0 -0.010544 rpy=-1.5708 0 -1.5708
- joint joint_link4_to_link5: axis 0.009166 0.999958 2.1e-05 -> 0 0 1; origin xyz=5.2e-05 0.0142 0.0325 rpy=0 0 0 -> xyz=0 -0.0142 0.0325 rpy=1.5708 -1.5708 0
- joint joint_link5_to_in_right_grip: axis -0.999947 0.009166 -0.004789 -> 0 0 1; origin xyz=0.002086 -0.000687 0.059134 rpy=0 0 0 -> xyz=0.059134 -0.002086 -0.000687 rpy=-1.5708 -0.17453 0
