Commit message: add end effector

File: urdf/cobot.description.xacro (robot description, xacro)
@@ -381,4 +381,5 @@
       </collision>
     </link>
+    <!-- joint -->
     <joint name="joint_base_link_to_link1" type="revolute">
       <origin
@@ -535,4 +536,15 @@
         effort="1000.0" lower="-1.5708" upper="1.5708" velocity="0.5" />
     </joint>
+    <!-- end effector -->
+    <link name="end_effector" />
+    <joint name="end_effector" type="fixed">
+      <origin
+        xyz="0.105 0 -0.0075"
+        rpy="0 0 0" />
+      <parent
+        link="link5" />
+      <child
+        link="end_effector" />
+    </joint>
   </xacro:macro>
 </robot>

File: urdf/cobot.urdf (robot description, URDF)
Before this commit: robot cobot, 7 links, 6 joints
Links:
- added link end_effector
- added link in_left_grip; collision mesh filename=package://cobot_description/meshes/in_left_grip.stl scale=0.001 0.001 0.001; visual mesh filename=package://cobot_description/meshes/in_left_grip.stl scale=0.001 0.001 0.001
- added link left_gripper; collision mesh filename=package://cobot_description/meshes/left_gripper.stl scale=0.001 0.001 0.001; visual mesh filename=package://cobot_description/meshes/left_gripper.stl scale=0.001 0.001 0.001
- added link out_left_grip; collision mesh filename=package://cobot_description/meshes/out_left_grip.stl scale=0.001 0.001 0.001; visual mesh filename=package://cobot_description/meshes/out_left_grip.stl scale=0.001 0.001 0.001
- added link out_right_grip; collision mesh filename=package://cobot_description/meshes/out_right_grip.stl scale=0.001 0.001 0.001; visual mesh filename=package://cobot_description/meshes/out_right_grip.stl scale=0.001 0.001 0.001
- added link right_gripper; collision mesh filename=package://cobot_description/meshes/right_gripper.stl scale=0.001 0.001 0.001; visual mesh filename=package://cobot_description/meshes/right_gripper.stl scale=0.001 0.001 0.001
- link in_right_grip: mass 0.020498186106830463 -> None
Joints:
- added joint end_effector: type fixed, parent link5, child end_effector, origin xyz=0.105 0 -0.0075 rpy=0 0 0
- added joint gripper: type revolute, parent link5, child out_left_grip, origin xyz=0.038208 0.00536837 -0.017277 rpy=-1.5708 0.2618 0, axis 0 0 -1, limit lower=-0.500 upper=0.250 effort=1000.0 velocity=0.5
- added joint joint_link5_to_in_left_grip: type revolute, parent link5, child in_left_grip, origin xyz=0.059059 -0.002086 -0.013997 rpy=-1.5708 0.34906 0, axis 0 0 -1, limit lower=-1.5708 upper=1.5708 effort=1000.0 velocity=0.5, mimic joint=gripper multiplier=1.2 offset=0
- added joint joint_link5_to_out_right_grip: type revolute, parent link5, child out_right_grip, origin xyz=0.038322 0.00536837 0.002815 rpy=-1.5708 -0.2618 0, axis 0 0 1, limit lower=-1.5708 upper=1.5708 effort=1000.0 velocity=0.5, mimic joint=gripper multiplier=1.0 offset=0
- added joint joint_out_left_grip_to_left_gripper: type revolute, parent out_left_grip, child left_gripper, origin xyz=0.0339442 0.00682491 -0.0042874 rpy=0 0 -0.5236, axis 0 0 1, limit lower=-1.5708 upper=1.5708 effort=1000.0 velocity=0.5, mimic joint=gripper multiplier=1.0 offset=0
- added joint joint_out_right_grip_to_right_gripper: type revolute, parent out_right_grip, child right_gripper, origin xyz=0.0339442 -0.00682491 -0.0030837 rpy=0 0 0.5236, axis 0 0 -1, limit lower=-1.5708 upper=1.5708 effort=1000.0 velocity=0.5, mimic joint=gripper multiplier=1.0 offset=0
- joint joint_base_link_to_link1: limit (none) -> lower=-1.5708 upper=1.5708 effort=1000.0 velocity=0.5; type continuous -> revolute
- joint joint_link1_to_link2: limit (none) -> lower=-1.5708 upper=1.5708 effort=1000.0 velocity=0.5; type continuous -> revolute
- joint joint_link2_to_link3: limit (none) -> lower=-1.5708 upper=1.5708 effort=1000.0 velocity=0.5; type continuous -> revolute
- joint joint_link3_to_link4: limit (none) -> lower=-1.5708 upper=1.5708 effort=1000.0 velocity=0.5; type continuous -> revolute
- joint joint_link4_to_link5: limit (none) -> lower=-1.5708 upper=1.5708 effort=1000.0 velocity=0.5; type continuous -> revolute
- joint joint_link5_to_in_right_grip: limit (none) -> lower=-1.5708 upper=1.5708 effort=1000.0 velocity=0.5; mimic (none) -> joint=gripper multiplier=1.2 offset=0; origin xyz=0.059134 -0.002086 -0.000687 rpy=-1.5708 -0.17453 0 -> xyz=0.059134 -0.002086 -0.000687 rpy=-1.5708 -0.34906 0; type continuous -> revolute

Commit message: modify gripper to open position

File: urdf/cobot.description.xacro (robot description, xacro)
@@ -451,5 +451,5 @@
       <origin
         xyz="0.038208 0.00536837 -0.017277"
-        rpy="-1.5708 0.2618 0"/>
+        rpy="-1.5708 1.047 0"/>
       <parent
         link="link5"/>
@@ -457,16 +457,76 @@
         link="out_left_grip"/>
       <axis
-         xyz="0 0 -1"/>
-      <limit
-        effort="1000.0" lower="-0.500" upper="0.250" velocity="0.5" />
+         xyz="0 0 1"/>
+      <limit
+        effort="1000.0" lower="-1.047" upper="0.0" velocity="0.5" />
     </joint>
     <joint name="joint_link5_to_out_right_grip" type="revolute">
       <origin
         xyz="0.038322 0.00536837 0.002815"
-        rpy="-1.5708 -0.2618 0"/>
+        rpy="-1.5708 -1.047 0"/>
       <parent
         link="link5"/>
       <child
         link="out_right_grip"/>
+      <axis
+        xyz="0 0 -1"/>
+      <mimic
+        joint="gripper" multiplier="1.0" offset="0" />
+      <limit
+        effort="1000.0" lower="-1.5708" upper="1.5708" velocity="0.5" />
+    </joint>
+    <joint name="joint_link5_to_in_left_grip" type="revolute">
+      <origin
+        xyz="0.059059 -0.002086 -0.013997"
+        rpy="-1.5708 1.3090 0" />
+      <parent
+        link="link5"/>
+      <child
+        link="in_left_grip"/>
+      <axis
+        xyz="0 0 1"/>
+      <mimic
+        joint="gripper" multiplier="1.2" offset="0" />
+      <limit
+        effort="1000.0" lower="-1.5708" upper="1.5708" velocity="0.5" />
+    </joint>
+    <joint name="joint_link5_to_in_right_grip" type="revolute">
+      <origin
+        xyz="0.059134 -0.002086 -0.000687"
+        rpy="-1.5708 -1.3090 0" />
+      <parent
+        link="link5" />
+      <child
+        link="in_right_grip" />
+      <axis
+        xyz="0 0 -1" />
+      <mimic
+        joint="gripper" multiplier="1.2" offset="0" />
+      <limit
+        effort="1000.0" lower="-1.5708" upper="1.5708" velocity="0.5" />
+    </joint>
+    <joint name="joint_out_left_grip_to_left_gripper" type="revolute">
+      <origin
+        xyz="0.0339442 0.00682491 -0.0042874"
+        rpy="0 0 -1.309" />
+      <parent
+        link="out_left_grip"/>
+      <child
+        link="left_gripper"/>
+      <axis
+        xyz="0 0 -1"/>
+      <mimic
+        joint="gripper" multiplier="1.0" offset="0" />
+      <limit
+        effort="1000.0" lower="-1.5708" upper="1.5708" velocity="0.5" />
+    </joint>
+    <joint name="joint_out_right_grip_to_right_gripper" type="revolute">
+      <origin
+        xyz="0.0339442 -0.00682491 -0.0030837"
+        rpy="0 0 1.309"/>
+      <parent
+        link="out_right_grip"/>
+      <child
+        link="right_gripper"/>
       <axis
         xyz="0 0 1"/>
@@ -476,64 +536,4 @@
         effort="1000.0" lower="-1.5708" upper="1.5708" velocity="0.5" />
     </joint>
-    <joint name="joint_link5_to_in_left_grip" type="revolute">
-      <origin
-        xyz="0.059059 -0.002086 -0.013997"
-        rpy="-1.5708 0.34906 0" />
-      <parent
-        link="link5"/>
-      <child
-        link="in_left_grip"/>
-      <axis
-        xyz="0 0 -1"/>
-      <mimic
-        joint="gripper" multiplier="1.2" offset="0" />
-      <limit
-        effort="1000.0" lower="-1.5708" upper="1.5708" velocity="0.5" />
-    </joint>
-    <joint name="joint_link5_to_in_right_grip" type="revolute">
-      <origin
-        xyz="0.059134 -0.002086 -0.000687"
-        rpy="-1.5708 -0.34906 0" />
-      <parent
-        link="link5" />
-      <child
-        link="in_right_grip" />
-      <axis
-        xyz="0 0 1" />
-      <mimic
-        joint="gripper" multiplier="1.2" offset="0" />
-      <limit
-        effort="1000.0" lower="-1.5708" upper="1.5708" velocity="0.5" />
-    </joint>
-    <joint name="joint_out_left_grip_to_left_gripper" type="revolute">
-      <origin
-        xyz="0.0339442 0.00682491 -0.0042874"
-        rpy="0 0 -0.5236" />
-      <parent
-        link="out_left_grip"/>
-      <child
-        link="left_gripper"/>
-      <axis
-        xyz="0 0 1"/>
-      <mimic
-        joint="gripper" multiplier="1.0" offset="0" />
-      <limit
-        effort="1000.0" lower="-1.5708" upper="1.5708" velocity="0.5" />
-    </joint>
-    <joint name="joint_out_right_grip_to_right_gripper" type="revolute">
-      <origin
-        xyz="0.0339442 -0.00682491 -0.0030837"
-        rpy="0 0 0.5236"/>
-      <parent
-        link="out_right_grip"/>
-      <child
-        link="right_gripper"/>
-      <axis
-        xyz="0 0 -1"/>
-      <mimic
-        joint="gripper" multiplier="1.0" offset="0" />
-      <limit
-        effort="1000.0" lower="-1.5708" upper="1.5708" velocity="0.5" />
-    </joint>
     <!-- end effector -->
     <link name="end_effector" />

File: urdf/cobot.urdf (robot description, URDF)
Before this commit: robot cobot, 13 links, 12 joints
Joints:
- joint gripper: origin xyz=0.038208 0.00536837 -0.017277 rpy=-1.5708 0.2618 0 -> xyz=0.038208 0.00536837 -0.017277 rpy=-1.5708 1.047 0
- joint joint_link5_to_in_left_grip: origin xyz=0.059059 -0.002086 -0.013997 rpy=-1.5708 0.34906 0 -> xyz=0.059059 -0.002086 -0.013997 rpy=-1.5708 1.3090 0
- joint joint_link5_to_in_right_grip: origin xyz=0.059134 -0.002086 -0.000687 rpy=-1.5708 -0.34906 0 -> xyz=0.059134 -0.002086 -0.000687 rpy=-1.5708 -1.3090 0
- joint joint_link5_to_out_right_grip: origin xyz=0.038322 0.00536837 0.002815 rpy=-1.5708 -0.2618 0 -> xyz=0.038322 0.00536837 0.002815 rpy=-1.5708 -1.047 0
- joint joint_out_left_grip_to_left_gripper: origin xyz=0.0339442 0.00682491 -0.0042874 rpy=0 0 -0.5236 -> xyz=0.0339442 0.00682491 -0.0042874 rpy=0 0 -1.309
- joint joint_out_right_grip_to_right_gripper: origin xyz=0.0339442 -0.00682491 -0.0030837 rpy=0 0 0.5236 -> xyz=0.0339442 -0.00682491 -0.0030837 rpy=0 0 1.309

Commit message: menyamakan nama joint di ros2_control dgn urdf xacro

File: urdf/cobot.description.xacro (robot description, xacro)
@@ -382,5 +382,5 @@
     </link>
     <!-- joint -->
-    <joint name="joint_base_link_to_link1" type="revolute">
+    <joint name="joint_0" type="revolute">
       <origin
         xyz="0 0 0.05675"
@@ -393,7 +393,7 @@
         xyz="0 0 1" />
       <limit
-        effort="1000.0" lower="-1.5708" upper="1.5708" velocity="0.5" />
-    </joint>
-    <joint name="joint_link1_to_link2" type="revolute">
+        effort="1000.0" lower="-1.57079632679" upper="1.57079632679" velocity="0.5" />
+    </joint>
+    <joint name="joint_1" type="revolute">
       <origin
         xyz="0.01392 0 0.070276"
@@ -406,7 +406,7 @@
         xyz="0 0 1" />
       <limit
-        effort="1000.0" lower="-1.5708" upper="1.5708" velocity="0.5" />
-    </joint>
-    <joint name="joint_link2_to_link3" type="revolute">
+        effort="1000.0" lower="-1.57079632679" upper="1.57079632679" velocity="0.5" />
+    </joint>
+    <joint name="joint_2" type="revolute">
       <origin
         xyz="0.12 0 0"
@@ -419,7 +419,7 @@
         xyz="0 0 -1"/>
       <limit
-        effort="1000.0" lower="-1.5708" upper="1.5708" velocity="0.5" />
-    </joint>
-    <joint name="joint_link3_to_link4" type="revolute">
+        effort="1000.0" lower="-1.57079632679" upper="1.57079632679" velocity="0.5" />
+    </joint>
+    <joint name="joint_3" type="revolute">
       <origin
         xyz="0.08975 0 -0.010544"
@@ -432,7 +432,7 @@
         xyz="0 0 1" />
       <limit
-        effort="1000.0" lower="-1.5708" upper="1.5708" velocity="0.5" />
-    </joint>
-    <joint name="joint_link4_to_link5" type="revolute">
+        effort="1000.0" lower="-1.57079632679" upper="1.57079632679" velocity="0.5" />
+    </joint>
+    <joint name="joint_4" type="revolute">
       <origin
         xyz="0 -0.0142 0.0325"
@@ -445,5 +445,5 @@
         xyz="0 0 1" />
       <limit
-        effort="1000.0" lower="-1.5708" upper="1.5708" velocity="0.5" />
+        effort="1000.0" lower="-1.57079632679" upper="1.57079632679" velocity="0.5" />
     </joint>
     <!-- joint_link5_to_out_left_grip -->
@@ -474,5 +474,5 @@
         joint="gripper" multiplier="1.0" offset="0" />
       <limit
-        effort="1000.0" lower="-1.5708" upper="1.5708" velocity="0.5" />
+        effort="1000.0" lower="-1.57079632679" upper="1.57079632679" velocity="0.5" />
     </joint>
     <joint name="joint_link5_to_in_left_grip" type="revolute">
@@ -489,5 +489,5 @@
         joint="gripper" multiplier="1.2" offset="0" />
       <limit
-        effort="1000.0" lower="-1.5708" upper="1.5708" velocity="0.5" />
+        effort="1000.0" lower="-1.57079632679" upper="1.57079632679" velocity="0.5" />
     </joint>
     <joint name="joint_link5_to_in_right_grip" type="revolute">
@@ -504,5 +504,5 @@
         joint="gripper" multiplier="1.2" offset="0" />
       <limit
-        effort="1000.0" lower="-1.5708" upper="1.5708" velocity="0.5" />
+        effort="1000.0" lower="-1.57079632679" upper="1.57079632679" velocity="0.5" />
     </joint>
     <joint name="joint_out_left_grip_to_left_gripper" type="revolute">
@@ -519,5 +519,5 @@
         joint="gripper" multiplier="1.0" offset="0" />
       <limit
-        effort="1000.0" lower="-1.5708" upper="1.5708" velocity="0.5" />
+        effort="1000.0" lower="-1.57079632679" upper="1.57079632679" velocity="0.5" />
     </joint>
     <joint name="joint_out_right_grip_to_right_gripper" type="revolute">
@@ -534,5 +534,5 @@
         joint="gripper" multiplier="1.0" offset="0" />
       <limit
-        effort="1000.0" lower="-1.5708" upper="1.5708" velocity="0.5" />
+        effort="1000.0" lower="-1.57079632679" upper="1.57079632679" velocity="0.5" />
     </joint>
     <!-- end effector -->
