Commit message: new but not ready yet

File: urdf/cobot.description.xacro (robot description, xacro)
@@ -1,14 +1,30 @@
-<?xml version="1.0" encoding="utf-8"?>
-<robot xmlns:xacro="https://www.ros.org/wiki/xacro">
-  <xacro:macro name="cobot_description">
-    <material name="silver">
-      <color rgba="0.7 0.7 0.7 1.0"/>
-    </material>
-    <!-- base_link -->
-    <link name="base_link">
-      <inertial>
-        <origin
-          xyz="0.0010569805350138673 0.0007297344522584362 0.01829217339489528"
-          rpy="0 0 0" />
+<?xml version="1.0" encoding="UTF-8"?>
+<robot xmlns:xacro="http://www.ros.org/wiki/xacro">
+  <xacro:include filename="$(find cobot_description)/urdf/utils/colors.xacro" />
+  <xacro:include filename="$(find cobot_description)/urdf/utils/inertials.xacro" />
+  <!-- simulation:=true membuang tag <mimic>, sehingga joint mimic dikendalikan
+       langsung oleh controller (gz_ros2_control tidak mendukung mimic dari URDF) -->
+  <xacro:macro name="cobot_description" params="simulation:=false">
+    <link name="world"/>
+    <joint name="world_to_base_link" type="fixed">
+      <parent link="world"/>
+      <child link="base_link"/>
+    </joint>
+    <link name="base_link" />
+    <joint name="base_link_to_base_bottom" type="fixed">
+      <parent link="base_link"/>
+      <child link="base_bottom"/>
+    </joint>
+    <!-- base_bottom -->
+    <link name="base_bottom">
+      <visual>
+        <origin xyz="0 0 0" rpy="0 0 0" />
+        <geometry>
+          <mesh filename="package://cobot_description/meshes/base_link.stl" scale="0.001 0.001 0.001" />
+        </geometry>
+        <material name="silver" />
+      </visual>
+      <inertial>
+        <origin xyz="0.0010569805350138673 0.0007297344522584362 0.01829217339489528" rpy="0 0 0" />
         <mass
           value="0.9757252027596308" />
@@ -21,35 +37,17 @@
           ixz="-0.0" />
       </inertial>
-      <visual>
-        <origin
-          xyz="0 0 0"
-          rpy="0 0 0" />
-        <geometry>
-          <mesh
-            filename="package://cobot_description/meshes/base_link.stl"
-            scale="0.001 0.001 0.001" />
-        </geometry>
-        <material
-          name="silver" />
-      </visual>
-      <collision>
-        <origin
-          xyz="0 0 0"
-          rpy="0 0 0" />
-        <geometry>
-          <mesh
-            filename="package://cobot_description/meshes/base_link.stl"
-            scale="0.001 0.001 0.001" />
-        </geometry>
-      </collision>
     </link>
     <!-- link1 -->
     <link name="link1">
-      <inertial>
-        <origin
-          xyz="-0.003818008823720768 0.008441513827613 0.03204494242786362"
-          rpy="0 0 0" />
-        <mass
-          value="0.8487763548317978" />
+      <visual>
+        <origin xyz="0 0 0" rpy="0 0 0" />
+        <geometry>
+          <mesh filename="package://cobot_description/meshes/link1.stl" scale="0.001 0.001 0.001" />
+        </geometry>
+        <material name="silver" />
+      </visual>
+      <inertial>
+        <origin xyz="-0.003818008823720768 0.008441513827613 0.03204494242786362" rpy="0 0 0" />
+        <mass value="0.85" />
         <inertia
           ixx="0.000968"
@@ -60,35 +58,17 @@
           ixz="-7.7e-05" />
       </inertial>
-      <visual>
-        <origin
-          xyz="0 0 0"
-          rpy="0 0 0" />
-        <geometry>
-          <mesh
-            filename="package://cobot_description/meshes/link1.stl"
-            scale="0.001 0.001 0.001" />
-        </geometry>
-        <material
-          name="silver" />
-      </visual>
-      <collision>
-        <origin
-          xyz="0 0 0"
-          rpy="0 0 0" />
-        <geometry>
-          <mesh
-            filename="package://cobot_description/meshes/link1.stl"
-            scale="0.001 0.001 0.001" />
-        </geometry>
-      </collision>
     </link>
     <!-- link2 -->
     <link name="link2">
-      <inertial>
-        <origin
-          xyz="0.06020229512696279 -0.002214238815772403 0.011894670876730499"
-          rpy="0 0 0" />
-        <mass
-          value="0.6612420873424198" />
+      <visual>
+        <origin xyz="0 0 0" rpy="0 0 0" />
+        <geometry>
+          <mesh filename="package://cobot_description/meshes/link2.stl" scale="0.001 0.001 0.001" />
+        </geometry>
+        <material name="silver" />
+      </visual>
+      <inertial>
+        <origin xyz="0.06020229512696279 -0.002214238815772403 0.011894670876730499" rpy="0 0 0" />
+        <mass value="0.65" />
         <inertia
           ixx="0.000127"
@@ -99,35 +79,17 @@
           ixz="1e-06" />
       </inertial>
-      <visual>
-        <origin
-          xyz="0 0 0"
-          rpy="0 0 0" />
-        <geometry>
-          <mesh
-            filename="package://cobot_description/meshes/link2.stl"
-            scale="0.001 0.001 0.001" />
-        </geometry>
-        <material
-          name="silver" />
-      </visual>
-      <collision>
-        <origin
-          xyz="0 0 0"
-          rpy="0 0 0" />
-        <geometry>
-          <mesh
-            filename="package://cobot_description/meshes/link2.stl"
-            scale="0.001 0.001 0.001" />
-        </geometry>
-      </collision>
     </link>
     <!-- link3 -->
     <link name="link3">
-      <inertial>
-        <origin
-          xyz="0.0409322245782118 -0.0006937756215695916 -0.008652145666434768"
-          rpy="0 0 0" />
-        <mass
-          value="0.4123818105357045" />
+      <visual>
+        <origin xyz="0 0 0" rpy="0 0 0" />
+        <geometry>
+          <mesh filename="package://cobot_description/meshes/link3.stl" scale="0.001 0.001 0.001" />
+        </geometry>
+        <material name="silver" />
+      </visual>
+      <inertial>
+        <origin xyz="0.0409322245782118 -0.0006937756215695916 -0.008652145666434768" rpy="0 0 0" />
+        <mass value="0.4" />
         <inertia
           ixx="8.7e-05"
@@ -138,34 +100,17 @@
           ixz="-5e-06" />
       </inertial>
-      <visual>
-        <origin
-          xyz="0 0 0"
-          rpy="0 0 0" />
-        <geometry>
-          <mesh
-            filename="package://cobot_description/meshes/link3.stl"
-            scale="0.001 0.001 0.001" />
-        </geometry>
-        <material name="silver" />
-      </visual>
-      <collision>
-        <origin
-          xyz="0 0 0"
-          rpy="0 0 0" />
-        <geometry>
-          <mesh
-            filename="package://cobot_description/meshes/link3.stl"
-            scale="0.001 0.001 0.001" />
-        </geometry>
-      </collision>
     </link>
     <!-- link4 -->
     <link name="link4">
-      <inertial>
-        <origin
-          xyz="0.0002076619932401616 -0.005563955264345595 0.02139744743586941"
-          rpy="0 0 0" />
-        <mass
-          value="0.1688382109185934" />
+      <visual>
+        <origin xyz="0 0 0" rpy="0 0 0" />
+        <geometry>
+          <mesh filename="package://cobot_description/meshes/link4.stl" scale="0.001 0.001 0.001" />
+        </geometry>
+        <material name="silver" />
+      </visual>
+      <inertial>
+        <origin xyz="0.0002076619932401616 -0.005563955264345595 0.02139744743586941" rpy="0 0 0" />
+        <mass value="0.17" />
         <inertia
           ixx="4.4e-05"
@@ -176,34 +121,9 @@
           ixz="-0.0" />
       </inertial>
-      <visual>
-        <origin
-          xyz="0 0 0"
-          rpy="0 0 0" />
-        <geometry>
-          <mesh
-            filename="package://cobot_description/meshes/link4.stl"
-            scale="0.001 0.001 0.001" />
-        </geometry>
-        <material
-          name="silver" />
-      </visual>
-      <collision>
-        <origin
-          xyz="0 0 0"
-          rpy="0 0 0" />
-        <geometry>
-          <mesh
-            filename="package://cobot_description/meshes/link4.stl"
-            scale="0.001 0.001 0.001" />
-        </geometry>
-      </collision>
     </link>
     <link name="link5">
       <inertial>
-        <origin
-          xyz="0.023252917458090605 0.0009180511930666074 -0.0026770648599710144"
-          rpy="1.5708 0 1.5708" />
-        <mass
-          value="0.17229950863980814" />
+        <origin xyz="0.023252917458090605 0.0009180511930666074 -0.0026770648599710144" rpy="1.5708 0 1.5708" />
+        <mass value="0.17" />
         <inertia
           ixx="9.6e-05"
@@ -215,335 +135,288 @@
       </inertial>
       <visual>
-        <origin
-          xyz="0 0 0"
-          rpy="0 0 0" />
-        <geometry>
-          <mesh
-            filename="package://cobot_description/meshes/link5.stl"
-            scale="0.001 0.001 0.001" />
-        </geometry>
-        <material
-          name="silver"/>
-      </visual>
-      <collision>
-        <origin
-          xyz="0 0 0"
-          rpy="0 0 0" />
-        <geometry>
-          <mesh
-            filename="package://cobot_description/meshes/link5.stl"
-            scale="0.001 0.001 0.001" />
-        </geometry>
-      </collision>
+        <origin xyz="0 0 0" rpy="0 0 0" />
+        <geometry>
+          <mesh filename="package://cobot_description/meshes/link5.stl" scale="0.001 0.001 0.001" />
+        </geometry>
+        <material name="silver"/>
+      </visual>
     </link>
     <link name="in_right_grip">
       <visual>
-        <origin
-          xyz="0 0 0"
-          rpy="0 0 0" />
-        <geometry>
-          <mesh
-            filename="package://cobot_description/meshes/in_right_grip.stl"
-            scale="0.001 0.001 0.001" />
-        </geometry>
-        <material
-          name="silver" />
-      </visual>
-      <collision>
-        <origin
-          xyz="0 0 0"
-          rpy="0 0 0" />
-        <geometry>
-          <mesh
-            filename="package://cobot_description/meshes/in_right_grip.stl"
-            scale="0.001 0.001 0.001" />
-        </geometry>
-      </collision>
+        <origin xyz="0 0 0" rpy="0 0 0" />
+        <geometry>
+          <mesh filename="package://cobot_description/meshes/in_right_grip.stl" scale="0.001 0.001 0.001" />
+        </geometry>
+        <material name="silver" />
+      </visual>
+      <collision>
+        <origin xyz="0.0149143 0 0.00349 " rpy="0 0 0" />
+        <geometry>
+          <box size="0.04 0.01 0.0168"/>
+        </geometry>
+      </collision>
+      <xacro:box_inertial
+        mass="0.005"
+        size="0.04 0.01 0.0168"
+        xyz="0.0149143 0 0.00349"
+        rpy="0 0 0" />
     </link>
     <link name="in_left_grip">
       <visual>
-        <origin
-          xyz="0 0 0"
-          rpy="0 0 0" />
-        <geometry>
-          <mesh
-            filename="package://cobot_description/meshes/in_left_grip.stl"
-            scale="0.001 0.001 0.001" />
-        </geometry>
-        <material
-          name="silver" />
-      </visual>
-      <collision>
-        <origin
-          xyz="0 0 0"
-          rpy="0 0 0" />
-        <geometry>
-          <mesh
-            filename="package://cobot_description/meshes/in_left_grip.stl"
-            scale="0.001 0.001 0.001" />
-        </geometry>
-      </collision>
+        <origin xyz="0 0 0" rpy="0 0 0" />
+        <geometry>
+          <mesh filename="package://cobot_description/meshes/in_left_grip.stl" scale="0.001 0.001 0.001" />
+        </geometry>
+        <material name="silver" />
+      </visual>
+      <collision>
+        <origin xyz="0.0149143 0 0.00349 " rpy="0 0 0" />
+        <geometry>
+          <box size="0.04 0.01 0.0168"/>
+        </geometry>
+      </collision>
+      <xacro:box_inertial
+        mass="0.005"
+        size="0.04 0.01 0.0168"
+        xyz="0.0149143 0 0.00349"
+        rpy="0 0 0" />
     </link>
     <link name="out_right_grip">
       <visual>
-        <origin
-          xyz="0 0 0"
-          rpy="0 0 0" />
-        <geometry>
-          <mesh
-            filename="package://cobot_description/meshes/out_right_grip.stl"
-            scale="0.001 0.001 0.001" />
-        </geometry>
-        <material
-          name="silver" />
-      </visual>
-      <collision>
-        <origin
-          xyz="0 0 0"
-          rpy="0 0 0" />
-        <geometry>
-          <mesh
-            filename="package://cobot_description/meshes/out_right_grip.stl"
-            scale="0.001 0.001 0.001" />
-        </geometry>
-      </collision>
+        <origin xyz="0 0 0" rpy="0 0 0" />
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
File: urdf/cobot.ros2_control.xacro (robot description, xacro)
@@ -1,47 +1,40 @@
 <?xml version="1.0" encoding="utf-8"?>
-<robot xmlns:xacro="https://www.ros.org/wiki/xacro">
-  <xacro:arg name="use_mock_components" default="false" />
-  <xacro:macro name="cobot_ros2_control">
+<robot xmlns:xacro="http://www.ros.org/wiki/xacro">
+  <xacro:macro name="cobot_ros2_control" params="use_real_hardware">
     <ros2_control name="cobot_ros2_control" type="system">
-      <xacro:if value="$(arg use_mock_components)">
+      <xacro:if value="${use_real_hardware}">
+        <hardware>
+          <plugin>cobot_hardware/CobotHardware</plugin>
+          <param name="port_name">/dev/esp32</param>
+          <param name="baud_rate">115200</param>
+        </hardware>
+      </xacro:if>
+      <xacro:unless value="${use_real_hardware}">
         <hardware>
           <plugin>mock_components/GenericSystem</plugin>
-        </hardware>
-      </xacro:if>
-      <xacro:unless value="$(arg use_mock_components)">
-        <hardware>
-          <plugin>cobot_hardware/CobotHardware</plugin>
-          <param name="port_name">/dev/esp32</param>  <!-- use udev rules! -->
-          <param name="baud_rate">115200</param>
         </hardware>
       </xacro:unless>
       <!-- joint -->
       <joint name="joint_0">
-        <param name="id">0</param>
         <command_interface name="position" />
         <state_interface name="position" />
       </joint>
       <joint name="joint_1">
-        <param name="id">1</param>
         <command_interface name="position" />
         <state_interface name="position" />
       </joint>
       <joint name="joint_2">
-        <param name="id">2</param>
         <command_interface name="position" />
         <state_interface name="position" />
       </joint>
       <joint name="joint_3">
-        <param name="id">3</param>
         <command_interface name="position" />
         <state_interface name="position" />
       </joint>
       <joint name="joint_4">
-        <param name="id">4</param>
         <command_interface name="position" />
         <state_interface name="position" />
       </joint>
-      <joint name="gripper">
-        <param name="id">5</param>
+      <joint name="joint_gripper">
         <command_interface name="position" />
         <state_interface name="position" />

File: urdf/cobot.urdf.xacro (robot description, xacro)
@@ -1,7 +1,9 @@
-<?xml version="1.0"?>
-<robot name="cobot" xmlns:xacro="https://www.ros.org/wiki/xacro">
+<?xml version="1.0" encoding="UTF-8"?>
+<robot name="cobot" xmlns:xacro="http://www.ros.org/wiki/xacro">
   <xacro:include filename="$(find cobot_description)/urdf/cobot.description.xacro" />
   <xacro:include filename="$(find cobot_description)/urdf/cobot.ros2_control.xacro" />
-  <xacro:cobot_description />
-  <xacro:cobot_ros2_control />
+  <xacro:arg name="simulation" default="true" />
+  <xacro:arg name="use_real_hardware" default="false" />
+  <xacro:cobot_description simulation="$(arg simulation)" />
+  <xacro:cobot_ros2_control use_real_hardware="$(arg use_real_hardware)" />
 </robot>
