Commit message: modify a little bit

File: gazebo/cobot.gazebo.urdf.xacro (robot description, xacro)
@@ -2,6 +2,6 @@
 <robot name="cobot" xmlns:xacro="https://www.ros.org/wiki/xacro">
   <xacro:include filename="$(find cobot_gazebo)/urdf/cobot.description.xacro" />
-  <xacro:include filename="$(find cobot_gazebo)/urdf/cobot.ros2_control.xacro" />
-  <xacro:include filename="$(find cobot_gazebo)/urdf/cobot.gazebo.xacro" />
+  <xacro:include filename="$(find cobot_gazebo)/gazebo/cobot.ros2_control.xacro" />
+  <xacro:include filename="$(find cobot_gazebo)/gazebo/cobot.gazebo.xacro" />
   <xacro:cobot_description />
   <xacro:cobot_ros2_control />

File: urdf/cobot.ros2_control.xacro (robot description, xacro)
@@ -25,5 +25,5 @@
         <state_interface name="position" />
       </joint>
-      <!-- <joint name="joint_3">
+      <joint name="joint_3">
         <param name="id">3</param>
         <command_interface name="position" />
@@ -35,10 +35,9 @@
         <state_interface name="position" />
       </joint>
-      <!- gripper ->
       <joint name="gripper">
         <param name="id">5</param>
         <command_interface name="position" />
         <state_interface name="position" />
-      </joint> -->
+      </joint>
     </ros2_control>
   </xacro:macro>
